File: ESP32/pcb1a/pcb1a.sch (EAGLE design)
At the start: 13 parts

Commit message: UPD: ESP32/pcb1a/
Parts:
- removed SV1: (no value), ytani1:PINHEAD-MA03-1
- removed SV2: (no value), ytani1:PINHEAD-MA02-1
- added GND, SW: (no value), ytani1:PINHEAD-MA01-1
- added R1, R2, R3: 10K, rcl:R-EU_0204/5
- SV9: device ytani1:PINHEAD-MA02-1 -> ytani1:PINHEAD-MA03-1
Connections:
- removed net N$5: SV2.2, SV3.4, SV9.2
- new net N$10: R1.1, SV6.1, SW.1
- net +3V3: now also R1.2, R2.1, R3.1; no longer SV1.2
- net GND: now also GND.1, SV9.2; no longer SV1.1
- net N$1: now also R3.2, SV3.3, SV9.1; no longer SV1.3, SV6.1
- net N$6: now also R2.2, SV3.4, SV9.3; no longer SV2.1, SV3.3, SV9.1
Other:
- moved on the sheet: SV3
