File: pcb1a/RotaryEncoder1.brd (EAGLE design)
At the start: 25.4 x 27 mm, 8 parts

Commit message: UPD: ESP32/pcb1a/
Parts:
- moved R2 0.64 mm to (15.2, 17.8)
- moved RE_G 0.64 mm to (10.2, 21.6)
- moved RE_SW 0.64 mm to (5.08, 21.6)
- moved SIG 0.64 mm to (17.8, 21.6)
- moved POW 0.63 mm to (17.8, 14.0)
- moved R1 0.63 mm to (15.2, 10.2)
- moved R3 0.63 mm to (12.7, 15.2)
- moved RE1 0.63 mm to (8.89, 5.08)
