File: ESP32/pcb1c/pcb1c.brd (EAGLE design)
At the start: 65 x 55 mm, 18 parts

Commit message: UPD: ESP32/pcb1c/
Parts:
- moved R1 22.7 mm to (58.4, 35.6), turned to 0 degrees
- moved BME280 18.0 mm to (57.1, 40.6), turned to 180 degrees
- moved SV9 18.0 mm to (54.6, 17.8)
- moved GND 13.0 mm to (57.1, 33.0)
- moved SW 13.0 mm to (52.1, 33.0)
- moved R3 9.86 mm to (58.4, 14.6), turned to 180 degrees
- moved P1 9.67 mm to (39.4, 50.8), turned to 0 degrees
- moved R2 7.43 mm to (58.4, 12.1), turned to 180 degrees
- moved CHG1 5.24 mm to (19.7, 45.7)
- moved OLED1 2.54 mm to (38.1, 22.9)
Routing:
- net GND: track 207.6 -> 181.9 mm, vias 0 -> 1
- net N$6: track 109.2 -> 88.9 mm
- net N$1: track 96.5 -> 78.7 mm, vias 0 -> 1
- net N$2: track 35.6 -> 53.3 mm
- net +3V3: track 174.0 -> 157.5 mm
- net N$10: track 71.1 -> 55.9 mm
- net N$3: track 40.6 -> 48.3 mm
- net N$5: track 38.9 -> 45.3 mm
- net N$11: track 4.92 -> 9.11 mm
Other:
- board size 65 x 55 mm -> 63.1 x 55 mm
