File: ESP32/pcb2/pcb1f.sch (EAGLE design)
At the start: 19 parts, among them P1 P1

Commit message: UPD: ESP32/pcb2/
Parts:
- removed USB1: USB1, ytani1:USB-C-DIRECT
- added U$1: AE-USB2.0-TYPE-C-CTRPB-1, ytani1:AE-USB2.0-TYPE-C-CTRPB-1
Connections:
- removed net VBUS: CD1.VIN, USB1.VBUS
- new net N$1: CD1.VIN, U$1.V+R
- net GND: now also U$1.V-R; no longer USB1.GND
Changed lines of the file:
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@@
 <part name="GND7" library="supply1" library_urn="urn:adsk.eagle:library:371" deviceset="GND" device=""/>
 <part name="CD1" library="ytani1" deviceset="MH-CD42" device=""/>
-<part name="USB1" library="ytani1" deviceset="USB-C-DIRECT" device="" value="USB1"/>
 <part name="GND9" library="supply1" library_urn="urn:adsk.eagle:library:371" deviceset="GND" device=""/>
 <part name="GND10" library="supply1" library_urn="urn:adsk.eagle:library:371" deviceset="GND" device=""/>
 <part name="GND8" library="supply1" library_urn="urn:adsk.eagle:library:371" deviceset="GND" device=""/>
+<part name="U$1" library="ytani1" deviceset="AE-USB2.0-TYPE-C-CTRPB-1" device=""/>
 </parts>
 <sheets>
@@
 <attribute name="VALUE" x="-58.42" y="63.5" size="1.778" layer="95"/>
 </instance>
-<instance part="USB1" gate="G$1" x="-76.2" y="68.58" smashed="yes">
-<attribute name="NAME" x="-81.28" y="80.01" size="1.778" layer="95"/>
-<attribute name="VALUE" x="-81.28" y="58.42" size="1.778" layer="96"/>
-</instance>
 <instance part="GND9" gate="1" x="-66.04" y="58.42" smashed="yes">
 <attribute name="VALUE" x="-68.58" y="55.88" size="1.778" layer="96"/>
@@
 <attribute name="VALUE" x="-63.5" y="83.82" size="1.778" layer="96"/>
 </instance>
+<instance part="U$1" gate="G$1" x="-86.36" y="73.66" smashed="yes"/>
 </instances>
 <busses>
@@
 <pinref part="GND9" gate="1" pin="GND"/>
 <wire x1="-66.04" y1="68.58" x2="-66.04" y2="60.96" width="0.1524" layer="91"/>
-<pinref part="USB1" gate="G$1" pin="GND"/>
 <pinref part="CD1" gate="G$1" pin="GNDVIN"/>
-<wire x1="-68.58" y1="73.66" x2="-66.04" y2="73.66" width="0.1524" layer="91"/>
 <wire x1="-66.04" y1="73.66" x2="-60.96" y2="73.66" width="0.1524" layer="91"/>
 <wire x1="-66.04" y1="68.58" x2="-66.04" y2="73.66" width="0.1524" layer="91"/>
 <junction x="-66.04" y="68.58"/>
-<junction x="-66.04" y="73.66"/>
+<pinref part="U$1" gate="G$1" pin="V-R"/>
+<wire x1="-76.2" y1="68.58" x2="-66.04" y2="68.58" width="0.1524" layer="91"/>
 </segment>
 <segment>
@@
 </segment>
 </net>
-<net name="VBUS" class="0">
-<segment>
-<pinref part="USB1" gate="G$1" pin="VBUS"/>
-<wire x1="-68.58" y1="76.2" x2="-60.96" y2="76.2" width="0.1524" layer="91"/>
-<pinref part="CD1" gate="G$1" pin="VIN"/>
-</segment>
-</net>
 <net name="BAT+" class="0">
 <segment>
@@
 </segment>
 </net>
+<net name="N$1" class="0">
+<segment>
+<pinref part="U$1" gate="G$1" pin="V+R"/>
+<pinref part="CD1" gate="G$1" pin="VIN"/>
+<wire x1="-76.2" y1="76.2" x2="-60.96" y2="76.2" width="0.1524" layer="91"/>
+</segment>
+</net>
