File: ESP32/pcb2/pcb1f.brd (EAGLE design)
At the start: 72 x 47 mm, 19 parts, among them P1 P1

Commit message: UPD: ESP32/pcb2/
Parts:
- removed USB1: USB1, ytani1:USB-C-DIRECT
- added U$1: AE-USB2.0-TYPE-C-CTRPB-1, ytani1:AE-USB2.0-TYPE-C-CTRPB-1
Connections:
- removed net VBUS: CD1.VIN, USB1.VBUS
- new net N$1: CD1.VIN, U$1.V_R
- net GND: now also U$1.GND_R; no longer USB1.GND
Routing:
- net N$1: track 0.00 -> 20.3 mm
- net VBUS: track 7.62 -> 0.00 mm
- net GND: track 153.4 -> 145.8 mm
Changed lines of the file:
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@@
 <element name="P1" library="ytani1" package="JST-PH2" package3d_urn="urn:adsk.eagle:package:23610139/1" value="P1" x="34.29" y="43.18" smashed="yes"/>
 <element name="CD1" library="ytani1" package="MH-CD42" value="MH-CD42" x="35.56" y="36.83" smashed="yes" rot="R180"/>
-<element name="USB1" library="ytani1" package="USB-C-DIRECT" value="USB1" x="11.43" y="57.15" smashed="yes"/>
+<element name="U$1" library="ytani1" package="AE-USB2.0-TYPE-C-CTRPB-1" value="AE-USB2.0-TYPE-C-CTRPB-1" x="12.7" y="38.1" smashed="yes"/>
 </elements>
 <signals>
@@
 <contactref element="CD1" pad="GNDBAT"/>
 <contactref element="CD1" pad="GND5V"/>
-<contactref element="USB1" pad="GND"/>
 <contactref element="CD1" pad="GNDVIN"/>
 <contactref element="P1" pad="2"/>
@@
 <wire x1="43.18" y1="43.18" x2="48.26" y2="38.1" width="0.6096" layer="1"/>
 <wire x1="25.4" y1="33.02" x2="22.86" y2="33.02" width="0.6096" layer="16"/>
-<wire x1="15.24" y1="43.18" x2="15.24" y2="40.64" width="0.6096" layer="16"/>
-<wire x1="5.08" y1="27.94" x2="5.08" y2="40.64" width="0.6096" layer="16"/>
-<wire x1="5.08" y1="40.64" x2="15.24" y2="40.64" width="0.6096" layer="16"/>
-<wire x1="15.24" y1="40.64" x2="22.86" y2="40.64" width="0.6096" layer="16"/>
-<wire x1="22.86" y1="40.64" x2="25.4" y2="40.64" width="0.6096" layer="16"/>
+<wire x1="5.08" y1="27.94" x2="5.08" y2="33.02" width="0.6096" layer="16"/>
 <wire x1="25.4" y1="38.1" x2="22.86" y2="38.1" width="0.6096" layer="16"/>
-<wire x1="22.86" y1="33.02" x2="22.86" y2="38.1" width="0.6096" layer="16"/>
-<wire x1="22.86" y1="38.1" x2="22.86" y2="40.64" width="0.6096" layer="16"/>
+<wire x1="22.86" y1="38.1" x2="22.86" y2="33.02" width="0.6096" layer="16"/>
+<wire x1="22.86" y1="33.02" x2="5.08" y2="33.02" width="0.6096" layer="16"/>
+<wire x1="25.4" y1="38.1" x2="25.4" y2="40.64" width="0.6096" layer="16"/>
+<contactref element="U$1" pad="GND_R"/>
+<wire x1="17.78" y1="38.1" x2="22.86" y2="38.1" width="0.6096" layer="16"/>
 </signal>
 <signal name="N$2">
@@
 <wire x1="60.96" y1="5.08" x2="60.96" y2="15.24" width="0.6096" layer="16"/>
 </signal>
-<signal name="VBUS">
-<contactref element="USB1" pad="VBUS"/>
-<contactref element="CD1" pad="VIN"/>
-<wire x1="25.4" y1="43.18" x2="17.78" y2="43.18" width="0.6096" layer="16"/>
-</signal>
 <signal name="BAT+">
 <contactref element="CD1" pad="BAT"/>
@@
 <wire x1="33.02" y1="43.18" x2="33.29" y2="43.18" width="0.6096" layer="16"/>
 </signal>
+<signal name="N$1">
+<contactref element="U$1" pad="V_R"/>
+<contactref element="CD1" pad="VIN"/>
+<wire x1="25.4" y1="43.18" x2="15.24" y2="43.18" width="0.6096" layer="16"/>
+<wire x1="15.24" y1="43.18" x2="15.24" y2="35.56" width="0.6096" layer="16"/>
+<wire x1="15.24" y1="35.56" x2="17.78" y2="35.56" width="0.6096" layer="16"/>
+</signal>
 </signals>

Commit message: UPD: ESP32/pcb2/
Parts:
- moved CD1 7.62 mm to (27.9, 36.8)
- moved U$1 5.68 mm to (10.2, 33.0), turned to 90 degrees
- moved BME280 2.54 mm to (55.9, 36.8)
Routing:
- net N$1: track 20.3 -> 10.2 mm
- net BAT+: track 15.5 -> 23.1 mm
- net +5V: track 22.1 -> 14.5 mm
- net N$3: track 45.7 -> 48.3 mm
- net N$2: track 45.7 -> 48.3 mm
- net GND: track 145.8 -> 148.3 mm
Other:
- board size 72 x 47 mm -> 71.4 x 45.7 mm
